Commit message: Imported upstream version '1.35.4' of 'upstream'

File: tiago_pro_description/ros2_control/ros2_control.urdf.xacro (robot description, xacro)
@@ -65,13 +65,52 @@
       </xacro:if>
     </xacro:if>
-  </xacro:macro>
-  <xacro:macro name="tiago_pro_ros2_control" params="use_sim_time:=^|false">
+    <xacro:if value="${has_teleop_arms}">
+        <xacro:ros2_control_arm name="arm_teleop_right_1" reduction="121.0" offset_value="${arm_right_1_joint_offset}" use_sea_transmission="${torque_estimation}" />
+        <xacro:ros2_control_arm name="arm_teleop_right_2" reduction="121.0" offset_value="${arm_right_2_joint_offset}" use_sea_transmission="${torque_estimation}" />
+        <xacro:ros2_control_arm name="arm_teleop_right_3" reduction="101.0" offset_value="${arm_right_3_joint_offset}" use_sea_transmission="${torque_estimation}" />
+        <xacro:ros2_control_arm name="arm_teleop_right_4" reduction="101.0" offset_value="${arm_right_4_joint_offset}" use_sea_transmission="${torque_estimation}" />
+        <xacro:ros2_control_arm name="arm_teleop_right_5" reduction="101.0" offset_value="${arm_right_5_joint_offset}" use_sea_transmission="${torque_estimation}" />
+        <xacro:ros2_control_arm name="arm_teleop_right_6" reduction="101.0" offset_value="${arm_right_6_joint_offset}" use_sea_transmission="${torque_estimation}" />
+        <xacro:ros2_control_arm name="arm_teleop_right_7" reduction="101.0" offset_value="${arm_right_7_joint_offset}" use_sea_transmission="${torque_estimation}" />
+        <xacro:ros2_control_arm name="arm_teleop_left_1" reduction="121.0" offset_value="${arm_left_1_joint_offset}" use_sea_transmission="${torque_estimation}" />
+        <xacro:ros2_control_arm name="arm_teleop_left_2" reduction="121.0" offset_value="${arm_left_2_joint_offset}" use_sea_transmission="${torque_estimation}" />
+        <xacro:ros2_control_arm name="arm_teleop_left_3" reduction="101.0" offset_value="${arm_left_3_joint_offset}" use_sea_transmission="${torque_estimation}" />
+        <xacro:ros2_control_arm name="arm_teleop_left_4" reduction="101.0" offset_value="${arm_left_4_joint_offset}" use_sea_transmission="${torque_estimation}" />
+        <xacro:ros2_control_arm name="arm_teleop_left_5" reduction="101.0" offset_value="${arm_left_5_joint_offset}" use_sea_transmission="${torque_estimation}" />
+        <xacro:ros2_control_arm name="arm_teleop_left_6" reduction="101.0" offset_value="${arm_left_6_joint_offset}" use_sea_transmission="${torque_estimation}" />
+        <xacro:ros2_control_arm name="arm_teleop_left_7" reduction="101.0" offset_value="${arm_left_7_joint_offset}" use_sea_transmission="${torque_estimation}" />
+        <xacro:if value="${has_teleop_ft_sensor_right}">
+          <xacro:include filename="$(find pal_urdf_utils)/urdf/ft_sensors/ftsensor.ros2_control.xacro"/>
+          <xacro:ros2_control_force_torque_sensor name="wrist_teleop_right_ft_sensor"/>
+        </xacro:if>
+        <xacro:if value="${has_teleop_ft_sensor_left}">
+          <xacro:include filename="$(find pal_urdf_utils)/urdf/ft_sensors/ftsensor.ros2_control.xacro"/>
+          <xacro:ros2_control_force_torque_sensor name="wrist_teleop_left_ft_sensor"/>
+        </xacro:if>
+        <xacro:if value="${end_effector_teleop_right == 'pal-pro-gripper'}">
+          <xacro:ros2_control_pal_pro_gripper name="gripper_teleop_right" reduction="1.0" />
+        </xacro:if>
+        <xacro:if value="${end_effector_teleop_left == 'pal-pro-gripper'}">
+          <xacro:ros2_control_pal_pro_gripper name="gripper_teleop_left" reduction="1.0" />
+        </xacro:if>
+    </xacro:if>
+  </xacro:macro>
+  <xacro:macro name="ros2_control_head_offset">
+    <!-- head -->
+    <xacro:ros2_control_head_joint name="head_1" reduction="1.0" offset_value="${head_1_joint_offset}" />
+    <xacro:ros2_control_head_joint name="head_2" reduction="1.0" offset_value="${head_2_joint_offset}" />
+  </xacro:macro>
+  <xacro:macro name="tiago_pro_ros2_control" params="use_sim_time:=^|false has_teleop_arms:=^|false">
     <xacro:arg name="arm_type_left" default="tiago-pro"/>
     <xacro:arg name="arm_type_right" default="tiago-pro"/>
     <xacro:arg name="end_effector_left" default="pal-pro-pripper"/>
     <xacro:arg name="end_effector_right" default="pal-pro-gripper"/>
+    <xacro:arg name="end_effector_teleop_left" default="no-end-effector"/>
+    <xacro:arg name="end_effector_teleop_right" default="no-end-effector"/>
     <xacro:arg name="ft_sensor_left" default="no-ft-sensor"/>
     <xacro:arg name="ft_sensor_right" default="no-ft-sensor"/>
-    <xacro:arg name="arm_calibration_dir" default="$(find tiago_pro_description)/urdf/calibration" />
+    <xacro:arg name="ft_sensor_teleop_left" default="no-ft-sensor"/>
+    <xacro:arg name="ft_sensor_teleop_right" default="no-ft-sensor"/>
+    <xacro:arg name="calibration_offset_dir" default="$(find tiago_pro_description)/urdf/calibration" />
     <!-- TODO-->
     <xacro:property name="arm_type_left" value="$(arg arm_type_left)" />
@@ -79,6 +118,10 @@
     <xacro:property name="end_effector_left" value="$(arg end_effector_left)" />
     <xacro:property name="end_effector_right" value="$(arg end_effector_right)" />
+    <xacro:property name="end_effector_teleop_left" value="$(arg end_effector_teleop_left)" />
+    <xacro:property name="end_effector_teleop_right" value="$(arg end_effector_teleop_right)" />
     <xacro:property name="has_ft_sensor_left" value="${ft_sensor_left != 'no-ft-sensor'}" />
     <xacro:property name="has_ft_sensor_right" value="${ft_sensor_right != 'no-ft-sensor'}" />
+    <xacro:property name="has_teleop_ft_sensor_left" value="${ft_sensor_teleop_left != 'no-ft-sensor'}" />
+    <xacro:property name="has_teleop_ft_sensor_right" value="${ft_sensor_teleop_right != 'no-ft-sensor'}" />
     <xacro:property name="has_arm_left" value="${arm_type_left != 'no-arm'}" />
     <xacro:property name="has_arm_right" value="${arm_type_right != 'no-arm'}" />
@@ -88,12 +131,12 @@
     <xacro:include filename="$(find tiago_pro_head_description)/urdf/head.ros2_control.xacro" />
     <xacro:include filename="$(find pal_sea_arm_description)/urdf/arm/arm.ros2_control.xacro" />
-    <xacro:if value="${end_effector_left == 'pal-pro-gripper' or end_effector_right == 'pal-pro-gripper'}">
+    <xacro:if value="${end_effector_left == 'pal-pro-gripper' or end_effector_right == 'pal-pro-gripper' or end_effector_teleop_left == 'pal-pro-gripper' or end_effector_teleop_right == 'pal-pro-gripper'}">
       <xacro:include filename="$(find pal_pro_gripper_description)/urdf/gripper.ros2_control.xacro" />
     </xacro:if>
-    <xacro:if value="${end_effector_left == 'allegro-hand' or end_effector_right == 'allegro-hand'}">
+    <xacro:if value="${end_effector_left == 'allegro-hand' or end_effector_right == 'allegro-hand' or end_effector_teleop_left == 'allegro-hand' or end_effector_teleop_right == 'allegro-hand'}">
       <xacro:include filename="$(find allegro_hand_description)/urdf/allegro_hand.ros2_control.xacro" />
     </xacro:if>
     <!-- calibration offsets -->
-    <xacro:include filename="$(arg arm_calibration_dir)/arm_calibration.urdf.xacro" />
+    <xacro:include filename="$(arg calibration_offset_dir)/calibration_offset.urdf.xacro" />
     <!-- Simulation -->
     <xacro:if value="$(arg use_sim_time)">
@@ -113,5 +156,5 @@
         <xacro:ros2_control_torso name="torso_lift" reduction="1.0" />
         <!-- head -->
-        <xacro:ros2_control_head />
+        <xacro:ros2_control_head_offset />
         <!-- arms -->
         <xacro:ros2_control_arms/>
@@ -123,4 +166,10 @@
           <xacro:ros2_control_allegro_hand name="gripper_left" pid_controllers="$(arg pid_controllers)" reduction="1.0" />
         </xacro:if>
+        <xacro:if value="${end_effector_teleop_right == 'allegro-hand'}">
+          <xacro:ros2_control_allegro_hand name="gripper_teleop_right" pid_controllers="$(arg pid_controllers)" reduction="1.0" />
+        </xacro:if>
+        <xacro:if value="${end_effector_teleop_left == 'allegro-hand'}">
+          <xacro:ros2_control_allegro_hand name="gripper_teleop_left" pid_controllers="$(arg pid_controllers)" reduction="1.0" />
+        </xacro:if>
       </ros2_control>
     </xacro:if>
@@ -143,5 +192,5 @@
         </hardware>
         <!-- head -->
-        <xacro:ros2_control_head />
+        <xacro:ros2_control_head_offset />
       </ros2_control>
       <!-- Ethercat system -->
@@ -152,4 +201,6 @@
           <param name="error_protection">true</param>
           <param name="idle_mode_on_stop">true</param>
+          <param name="expose_collision_interface">true</param>
+          <param name="expose_safety_interface">true</param>
         </hardware>
         <!-- arms -->
@@ -164,4 +215,11 @@
         <xacro:allegro_ros2_control side="left" allegro_can="can1" pid_controllers="$(arg pid_controllers)"/>
       </xacro:if>
+      <!-- To test! -->
+      <!-- <xacro:if value="${end_effector_teleop_right == 'allegro-hand'}">
+        <xacro:allegro_ros2_control side="right" allegro_can="can2" pid_controllers="$(arg pid_controllers)"/>
+      </xacro:if>
+      <xacro:if value="${end_effector_teleop_left == 'allegro-hand'}">
+        <xacro:allegro_ros2_control side="left" allegro_can="can1" pid_controllers="$(arg pid_controllers)"/>
+      </xacro:if> -->
     </xacro:unless>
   </xacro:macro>

Commit message: Imported upstream version '2.4.1' of 'upstream'

File: tiago_pro_description/robots/tiago_pro.urdf.xacro (robot description, xacro)
@@ -12,5 +12,5 @@
   limitations under the License.
 -->
-<robot xmlns:xacro="http://ros.org/wiki/xacro" name="tiago_pro">
+<robot xmlns:xacro="http://ros.org/wiki/xacro" xmlns:gz="http://gazebosim.org/schema" name="tiago_pro">
   <!-- ARGUMENTS -->
   <!-- no-laser, sick-571-->
@@ -52,6 +52,8 @@
   <!-- no-ft-sensor, rokubi -->
   <xacro:arg name="ft_sensor_teleop_right" default="no-ft-sensor" />
-  <!-- realsense-d435 -->
-  <xacro:arg name="camera_model" default="realsense-d435" />
+  <!-- realsense-d435i -->
+  <xacro:arg name="camera_model" default="realsense-d435i" />
+  <!-- limits v2 -->
+  <xacro:arg name="limits_v2" default="False" />
   <!-- False, True -->
   <xacro:arg name="torque_estimation" default="False" />
@@ -73,4 +75,5 @@
   <xacro:arg name="arm_pitch" default="0.0" />
   <xacro:arg name="arm_yaw" default="-1.2217" />
+  <xacro:arg name="wheel_model" default="moog" />
   <!-- PROPERTIES -->
   <xacro:property name="torque_estimation" value="$(arg torque_estimation)" />
@@ -119,4 +122,5 @@
   <xacro:property name="end_effector_teleop_left_link" value="${'wrist_teleop_left_ft_tool_link' if has_teleop_ft_sensor_left else 'arm_teleop_left_tool_link'}" />
   <xacro:property name="end_effector_right_name" value="gripper_right" />
+  <xacro:property name="limits_v2" value="$(arg limits_v2)" />
   <xacro:property name="has_end_effector_teleop_left" value="${end_effector_teleop_left not in ['no-end-effector']}" />
   <xacro:property name="has_end_effector_teleop_right" value="${end_effector_teleop_right not in ['no-end-effector']}" />
@@ -124,4 +128,5 @@
   <xacro:property name="end_effector_teleop_right_name" value="gripper_teleop_right" />
   <xacro:property name="has_wrist_camera" value="$(arg has_wrist_camera)" />
+  <xacro:property name="wheel_model" value="$(arg wheel_model)" />
   <!-- Properties check -->
   <xacro:if value="${arm_type_left not in ['tiago-pro-prototype', 'tiago-pro', 'tiago-pro-s', 'no-arm']}">
@@ -163,4 +168,7 @@
   <xacro:if value="${laser_model not in ['no-laser', 'sick-571']}">
     <xacro:wrong_laser_model />
+  </xacro:if>
+  <xacro:if value="${wheel_model not in ['moog', 'grassland', 'no-wheels']}">
+    <xacro:wrong_wheel_model />
   </xacro:if>
   <!-- Compatibility check within TC and ft sensors-->
@@ -254,5 +262,5 @@
   <xacro:if value="${has_arm_left}">
     <!-- Arm -->
-    <xacro:pal_sea_arm name="arm_left" parent="torso_lift_link" arm_type="${arm_type_left}" wrist_model="${wrist_model_left}" tool_changer="${tool_changer_left}" reflect="1" joint_reflect="-1" arm_1_offset="${arm_left_1_joint_offset}" arm_2_offset="${arm_left_2_joint_offset}" arm_3_offset="${arm_left_3_joint_offset}" arm_4_offset="${arm_left_4_joint_offset}" arm_5_offset="${arm_left_5_joint_offset}" arm_6_offset="${arm_left_6_joint_offset}" arm_7_offset="${arm_left_7_joint_offset}">
+    <xacro:pal_sea_arm name="arm_left" parent="torso_lift_link" arm_type="${arm_type_left}" wrist_model="${wrist_model_left}" tool_changer="${tool_changer_left}" reflect="1" joint_reflect="-1" arm_1_offset="${arm_left_1_joint_offset}" arm_2_offset="${arm_left_2_joint_offset}" arm_3_offset="${arm_left_3_joint_offset}" arm_4_offset="${arm_left_4_joint_offset}" arm_5_offset="${arm_left_5_joint_offset}" arm_6_offset="${arm_left_6_joint_offset}" arm_7_offset="${arm_left_7_joint_offset}" limits_v2="${limits_v2}">
       <origin xyz="$(arg arm_x) $(arg arm_y) $(arg arm_z)" rpy="$(arg arm_roll) $(arg arm_pitch) $(arg arm_yaw)"/>
     </xacro:pal_sea_arm>
@@ -262,5 +270,5 @@
     </xacro:if>
     <xacro:if value="${has_wrist_camera}">
-      <xacro:pal_sea_arm_end_effector_camera name="gripper_left" parent="${end_effector_left_link}" type="realsense-d435" camera_position="up"/>
+      <xacro:pal_sea_arm_end_effector_camera name="gripper_left" parent="${end_effector_left_link}" type="realsense-d435i" camera_position="up"/>
     </xacro:if>
     <!-- FT sensors -->
@@ -272,5 +280,5 @@
   <xacro:if value="${has_arm_right}">
     <!-- Arm -->
-    <xacro:pal_sea_arm name="arm_right" parent="torso_lift_link" arm_type="${arm_type_right}" wrist_model="${wrist_model_right}" tool_changer="${tool_changer_right}" reflect="1" joint_reflect="1" arm_1_offset="${arm_right_1_joint_offset}" arm_2_offset="${arm_right_2_joint_offset}" arm_3_offset="${arm_right_3_joint_offset}" arm_4_offset="${arm_right_4_joint_offset}" arm_5_offset="${arm_right_5_joint_offset}" arm_6_offset="${arm_right_6_joint_offset}" arm_7_offset="${arm_right_7_joint_offset}">
+    <xacro:pal_sea_arm name="arm_right" parent="torso_lift_link" arm_type="${arm_type_right}" wrist_model="${wrist_model_right}" tool_changer="${tool_changer_right}" reflect="1" joint_reflect="1" arm_1_offset="${arm_right_1_joint_offset}" arm_2_offset="${arm_right_2_joint_offset}" arm_3_offset="${arm_right_3_joint_offset}" arm_4_offset="${arm_right_4_joint_offset}" arm_5_offset="${arm_right_5_joint_offset}" arm_6_offset="${arm_right_6_joint_offset}" arm_7_offset="${arm_right_7_joint_offset}" limits_v2="${limits_v2}">
       <origin xyz="$(arg arm_x) ${-1.0*$(arg arm_y)} $(arg arm_z)" rpy="$(arg arm_roll) ${-1.0*$(arg arm_pitch)} ${-3.14159 -$(arg arm_yaw)}"/>
     </xacro:pal_sea_arm>
@@ -280,5 +288,5 @@
     </xacro:if>
     <xacro:if value="${has_wrist_camera}">
-      <xacro:pal_sea_arm_end_effector_camera name="gripper_right" parent="${end_effector_right_link}" type="realsense-d435" camera_position="up"/>
+      <xacro:pal_sea_arm_end_effector_camera name="gripper_right" parent="${end_effector_right_link}" type="realsense-d435i" camera_position="up"/>
     </xacro:if>
     <!-- FT sensors -->
@@ -315,4 +323,4 @@
   </xacro:if>
   <!-- ROS 2 Control -->
-  <xacro:tiago_pro_ros2_control use_sim_time="$(arg use_sim_time)" has_teleop_arms="${has_teleop_arms}"/>
+  <xacro:tiago_pro_ros2_control use_sim_time="$(arg use_sim_time)" has_teleop_arms="${has_teleop_arms}" gazebo_version="${gazebo_version}"/>
 </robot>

File: tiago_pro_description/ros2_control/ros2_control.urdf.xacro (robot description, xacro)
@@ -37,6 +37,8 @@
       <xacro:ros2_control_arm name="arm_left_4" reduction="101.0" offset_value="${arm_left_4_joint_offset}" use_sea_transmission="${torque_estimation}" />
       <xacro:ros2_control_arm name="arm_left_5" reduction="101.0" offset_value="${arm_left_5_joint_offset}" use_sea_transmission="${torque_estimation}" />
-      <xacro:ros2_control_arm name="arm_left_6" reduction="101.0" offset_value="${arm_left_6_joint_offset}" use_sea_transmission="${torque_estimation}" />
-      <xacro:ros2_control_arm name="arm_left_7" reduction="101.0" offset_value="${arm_left_7_joint_offset}" use_sea_transmission="${torque_estimation}" />
+      <xacro:if value="${wrist_model_left != 'short-wrist'}">
+        <xacro:ros2_control_arm name="arm_left_6" reduction="101.0" offset_value="${arm_left_6_joint_offset}" use_sea_transmission="${torque_estimation}" />
+        <xacro:ros2_control_arm name="arm_left_7" reduction="101.0" offset_value="${arm_left_7_joint_offset}" use_sea_transmission="${torque_estimation}" />
+      </xacro:if>
       <xacro:if value="${has_ft_sensor_left}">
         <xacro:include filename="$(find pal_urdf_utils)/urdf/ft_sensors/ftsensor.ros2_control.xacro"/>
@@ -54,6 +56,8 @@
       <xacro:ros2_control_arm name="arm_right_4" reduction="101.0" offset_value="${arm_right_4_joint_offset}" use_sea_transmission="${torque_estimation}" />
       <xacro:ros2_control_arm name="arm_right_5" reduction="101.0" offset_value="${arm_right_5_joint_offset}" use_sea_transmission="${torque_estimation}" />
-      <xacro:ros2_control_arm name="arm_right_6" reduction="101.0" offset_value="${arm_right_6_joint_offset}" use_sea_transmission="${torque_estimation}" />
-      <xacro:ros2_control_arm name="arm_right_7" reduction="101.0" offset_value="${arm_right_7_joint_offset}" use_sea_transmission="${torque_estimation}" />
+      <xacro:if value="${wrist_model_right != 'short-wrist'}">
+        <xacro:ros2_control_arm name="arm_right_6" reduction="101.0" offset_value="${arm_right_6_joint_offset}" use_sea_transmission="${torque_estimation}" />
+        <xacro:ros2_control_arm name="arm_right_7" reduction="101.0" offset_value="${arm_right_7_joint_offset}" use_sea_transmission="${torque_estimation}" />
+      </xacro:if>
       <xacro:if value="${has_ft_sensor_right}">
         <xacro:include filename="$(find pal_urdf_utils)/urdf/ft_sensors/ftsensor.ros2_control.xacro"/>
@@ -101,5 +105,5 @@
     <xacro:ros2_control_head_joint name="head_2" reduction="1.0" offset_value="${head_2_joint_offset}" />
   </xacro:macro>
-  <xacro:macro name="tiago_pro_ros2_control" params="use_sim_time:=^|false has_teleop_arms:=^|false">
+  <xacro:macro name="tiago_pro_ros2_control" params="use_sim_time:=^|false has_teleop_arms:=^|false gazebo_version:=^|classic">
     <xacro:arg name="arm_type_left" default="tiago-pro"/>
     <xacro:arg name="arm_type_right" default="tiago-pro"/>
@@ -112,4 +116,5 @@
     <xacro:arg name="ft_sensor_teleop_left" default="no-ft-sensor"/>
     <xacro:arg name="ft_sensor_teleop_right" default="no-ft-sensor"/>
+    <xacro:arg name="wheel_model" default="moog"/>
     <xacro:arg name="calibration_offset_dir" default="$(find tiago_pro_description)/urdf/calibration" />
     <!-- TODO-->
@@ -127,4 +132,5 @@
     <xacro:property name="has_arm_right" value="${arm_type_right != 'no-arm'}" />
     <xacro:property name="can_device_name" value="can_device" />
+    <xacro:property name="wheel_model" value="$(arg wheel_model)" />
     <xacro:include filename="$(find omni_base_description)/urdf/wheels/wheel.ros2_control.xacro" />
     <xacro:include filename="$(find tiago_pro_description)/urdf/torso/torso.ros2_control.xacro" />
@@ -143,11 +149,25 @@
       <!-- Init the ROS 2 control gazebo interface -->
       <gazebo>
-        <plugin filename="libgazebo_ros2_control.so" name="gazebo_ros2_control">
-          <parameters>$(find tiago_pro_description)/ros2_control/gazebo_controller_manager_cfg.yaml</parameters>
-        </plugin>
+        <xacro:if value="${gazebo_version == 'classic'}">
+          <plugin filename="libgazebo_ros2_control.so" name="gazebo_ros2_control">
+            <parameters>$(find tiago_pro_description)/ros2_control/gazebo_controller_manager_cfg.yaml</parameters>
+          </plugin>
+        </xacro:if>
+        <xacro:if value="${gazebo_version == 'gazebo'}">
+          <plugin filename="gz_ros2_control-system" name="gz_ros2_control::GazeboSimROS2ControlPlugin">
+            <robot_param>robot_description</robot_param>
+            <robot_param_node>robot_state_publisher</robot_param_node>
+            <parameters>$(find tiago_pro_description)/ros2_control/gazebo_controller_manager_cfg.yaml</parameters>
+          </plugin>
+        </xacro:if>
       </gazebo>
       <ros2_control name="ros2_control_gazebo_system" type="system">
         <hardware>
-          <plugin>gazebo_ros2_control/GazeboSystem</plugin>
+          <xacro:if value="${gazebo_version == 'classic'}">
+            <plugin>gazebo_ros2_control/GazeboSystem</plugin>
+          </xacro:if>
+          <xacro:if value="${gazebo_version == 'gazebo'}">
+            <plugin>gz_ros2_control/GazeboSimSystem</plugin>
+          </xacro:if>
         </hardware>
         <!-- wheels -->
@@ -176,13 +196,16 @@
     <!-- Hardware -->
     <xacro:unless value="$(arg use_sim_time)">
-      <!-- CAN system -->
-      <ros2_control name="ros2_control_tiago_pro_system_can" type="system" rw_rate="100">
-        <hardware>
-          <plugin>robot_control/RobotControl</plugin>
-          <param name="group">can</param>
-        </hardware>
-        <!-- wheels -->
-        <xacro:ros2_control_wheels />
-      </ros2_control>
+      <xacro:if value="${wheel_model == 'moog'}">
+        <!-- CAN system -->
+        <ros2_control name="ros2_control_tiago_pro_system_can" type="system" rw_rate="100">
+          <!-- Execution env config -->
+          <hardware>
+            <plugin>robot_control/RobotControl</plugin>
+            <param name="group">can</param>
+          </hardware>
+          <!-- wheels -->
+          <xacro:ros2_control_wheels />
+        </ros2_control>
+      </xacro:if>
       <!-- Dynamixels system -->
       <ros2_control name="ros2_control_tiago_pro_system_dynamixel" type="system" rw_rate="100">
@@ -206,5 +229,10 @@
         <!-- arms -->
         <xacro:ros2_control_arms/>
+        <!-- torso -->
         <xacro:ros2_control_torso name="torso_lift" reduction="1.0" />
+        <xacro:if value="${wheel_model == 'grassland'}">
+          <!-- wheels -->
+          <xacro:ros2_control_wheels />
+        </xacro:if>
       </ros2_control>
       <xacro:arg name="pid_controllers" default="true"/>
